Commit message: Fixed problem in lookupTransform params. Using tf for joint positions still doesn't work. Going to try using joint_state topic

File: model/kuka1.urdf (robot description, URDF)
Before this commit: robot kuka_lwr, 9 links, 8 joints
Links:
- removed link world
- added link base_link
Joints:
- joint base_joint: parent world -> base_link

Commit message: Init position error solved and reduced duration to half

File: model/kuka1.urdf (robot description, URDF)
Before this commit: robot kuka_lwr, 9 links, 8 joints
Links:
- removed link base_link
- added link world
Joints:
- joint base_joint: parent base_link -> world
